Commit message: only urdf LTS

File: description/jannik.xacro (robot description, xacro)
@@ -196,12 +196,3 @@
         </inertial>
     </link>
-    <!-- A simple fixed joint from our empty world link, to our base. -->
-    <!-- The base origin is offset from the world origin. -->
-    <joint name="base_joint_2" type="prismatic">
-        <origin xyz="0 0 -0.1" rpy="0 0 0"/>
-        <parent link="world"/>
-        <child link="front_foot"/>
-        <axis xyz="1 0 0"/>
-        <limit lower="-2" upper="2" velocity="100" effort="100"/>
-    </joint>
 </robot>

File: description/jannik_first.xacro (robot description, xacro)
@@ -109,5 +109,5 @@
             <origin xyz="1 0 0.15" rpy="0 0 0"/>
             <geometry>
-                <box size="0.3 0.3 2" />
+                <box size="2 0.3 0.3" />
             </geometry>
         </collision>
