Commit message: gazebo spown

File: description/jannik copy.xacro (robot description, xacro)
@@ -8,11 +8,4 @@
     <!-- This first link called "world" is empty -->
     <link name="world"></link>
-    <!-- A simple fixed joint from our empty world link, to our base. -->
-    <!-- The base origin is offset from the world origin. -->
-    <joint name="base_joint" type="fixed">
-        <origin xyz="0 0 0" rpy="0 0 0"/>
-        <parent link="world"/>
-        <child link="back_foot"/>
-    </joint>
     <!-- base_link is a large rectangular plate. Some things to note: -->
     <!-- - We set the visual origin Z to half the box height, so that the link origin sits at the bottom of the box -->
@@ -26,5 +19,5 @@
                 <box size="1 0.5 0.2" />
             </geometry>
-            <material name="green">
+            <material name="white">
                 <color rgba="0.2 1 0.2 1"/>
             </material>
@@ -64,5 +57,5 @@
                 <box size="0.3 0.3 2" />
             </geometry>
-            <material name="green">
+            <material name="orange">
                 <color rgba="0.2 1 0.2 1"/>
             </material>
@@ -109,5 +102,5 @@
             <origin xyz="1 0 0.15" rpy="0 0 0"/>
             <geometry>
-                <box size="2 0.3 0.3" />
+                <box size="0.3 0.3 2" />
             </geometry>
         </collision>
@@ -140,5 +133,5 @@
                 <box size="0.3 0.3 2" />
             </geometry>
-            <material name="green">
+            <material name="orange">
                 <color rgba="0.2 1 0.2 1"/>
             </material>
@@ -178,5 +171,5 @@
                 <box size="1 0.5 0.2" />
             </geometry>
-            <material name="green">
+            <material name="white">
                 <color rgba="0.2 1 0.2 1"/>
             </material>
